Commit message: remove unnecessary files

File: crane_x7_description/urdf/camera.urdf (robot description, URDF)
Before this commit: robot camera, 1 links, 1 joints
Joints:
- joint camera_joint: origin xyz=0 0.1 0 rpy=0 1.570796326795 0 -> xyz=0 0.1 0 rpy=0 4.7123889803846898576939650749193 0

File: crane_x7_description/urdf/crane_x7.xacro (robot description, xacro)
@@ -1,8 +1,8 @@
 <?xml version="1.0"?>
+<!--This file is changed by group8 -->
 <robot xmlns:xacro="http://ros.org/wiki/xacro">
   <xacro:include filename="$(find crane_x7_description)/urdf/crane_x7_mounting_plate.xacro"/>
   <xacro:include filename="$(find crane_x7_description)/urdf/crane_x7_arm.xacro"/>
   <xacro:include filename="$(find crane_x7_description)/urdf/crane_x7_wide_two_finger_gripper.xacro"/>
-  <!--追加！！！-->
   <xacro:include filename="$(find crane_x7_description)/urdf/camera.urdf"/>
   <material name="black">
